File: rp2040.kicad_sch (KiCad schematic)
At the start: 35 parts, among them J3 USB_B_Micro, SW1 SW_Push, SW2 SW_Push, U1 RP2040, U2 TPUSBLC6-4SC6, U3 NCP1117-3.3_SOT223, U4 FM25W32, Y1 Crystal_GND24

Commit message: improvements
Parts:
- C14: renamed from C2; footprint Capacitor_SMD:C_0402_1005Metric_Pad0.74x0.62mm_HandSolder -> Capacitor_SMD:C_0603_1608Metric_Pad1.08x0.95mm_HandSolder
- C17: renamed from C12; footprint Capacitor_SMD:C_0402_1005Metric_Pad0.74x0.62mm_HandSolder -> Capacitor_SMD:C_0603_1608Metric_Pad1.08x0.95mm_HandSolder
- J1: renamed from J3; footprint footprints:DEALON USB-MR-D-037 -> rp2040-core:DEALON USB-MR-D-037
- SW73: renamed from SW2; footprint footprints:BZCN TSC003A0826A -> rp2040-core:BZCN TSC003A0826A
- SW74: renamed from SW1; footprint footprints:BZCN TSC003A0826A -> rp2040-core:BZCN TSC003A0826A
- renumbered C17 to C10, C16 to C11, C14 to C12, C15 to C13, C9 to C15, C11 to C16, C5 to C18, C6 to C19, C1 to C3, C3 to C4, C4 to C5, C7 to C6, C8 to C7, C10 to C8, C13 to C9, D1 to D75, R6 to R10, R5 to R11, R3 to R12, R4 to R13, R2 to R14, R1 to R15, R8 to R16, R7 to R9, U3 to U2, U2 to U3, U1 to U5, Y1 to Y2
Connections:
- net MCU_USB_D+: now reaches R13.2, U5.47 (USB_DP)
- net MCU_USB_D-: now reaches R14.2, U5.46 (USB_DM)
Other:
- moved on the sheet: R13, R14

Commit message: relinked the footprints
Parts:
- C10, C11, C12, C13, C15, C16, C18, C19, C3, C4, C5, C6, C7, C8, C9: footprint Capacitor_SMD:C_0402_1005Metric_Pad0.74x0.62mm_HandSolder -> Capacitor_SMD:C_0402_1005Metric
- C14, C17: footprint Capacitor_SMD:C_0603_1608Metric_Pad1.08x0.95mm_HandSolder -> Capacitor_SMD:C_0603_1608Metric
- D75: footprint LED_SMD:LED_0603_1608Metric_Pad1.05x0.95mm_HandSolder -> LED_SMD:LED_0603_1608Metric
- FB1, R10, R11, R12, R13, R14, R15, R16, R9: footprint Resistor_SMD:R_0402_1005Metric_Pad0.72x0.64mm_HandSolder -> Resistor_SMD:R_0402_1005Metric
Changed lines of the file:
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@@
       (effects (font (size 1.27 1.27)) (justify left))
     )
-    (property "Footprint" "Capacitor_SMD:C_0402_1005Metric_Pad0.74x0.62mm_HandSolder" (id 2) (at 126.6952 52.07 0)
+    (property "Footprint" "Capacitor_SMD:C_0402_1005Metric" (id 2) (at 126.6952 52.07 0)
       (effects (font (size 1.27 1.27)) hide)
     )
@@
       (effects (font (size 1.27 1.27)) (justify left))
     )
-    (property "Footprint" "Capacitor_SMD:C_0402_1005Metric_Pad0.74x0.62mm_HandSolder" (id 2) (at 91.1352 52.07 0)
+    (property "Footprint" "Capacitor_SMD:C_0402_1005Metric" (id 2) (at 91.1352 52.07 0)
       (effects (font (size 1.27 1.27)) hide)
     )
@@
       (effects (font (size 1.27 1.27)) (justify left))
     )
-    (property "Footprint" "Capacitor_SMD:C_0402_1005Metric_Pad0.74x0.62mm_HandSolder" (id 2) (at 387.6802 57.15 0)
+    (property "Footprint" "Capacitor_SMD:C_0402_1005Metric" (id 2) (at 387.6802 57.15 0)
       (effects (font (size 1.27 1.27)) hide)
     )
@@
     (property "Reference" "R13" (id 0) (at 80.645 171.45 90))
     (property "Value" "27.4" (id 1) (at 80.645 173.99 90))
-    (property "Footprint" "Resistor_SMD:R_0402_1005Metric_Pad0.72x0.64mm_HandSolder" (id 2) (at 80.645 179.578 90)
+    (property "Footprint" "Resistor_SMD:R_0402_1005Metric" (id 2) (at 80.645 179.578 90)
       (effects (font (size 1.27 1.27)) hide)
     )
@@
       (effects (font (size 1.27 1.27)) (justify left))
     )
-    (property "Footprint" "Capacitor_SMD:C_0402_1005Metric_Pad0.74x0.62mm_HandSolder" (id 2) (at 45.4152 52.07 0)
+    (property "Footprint" "Capacitor_SMD:C_0402_1005Metric" (id 2) (at 45.4152 52.07 0)
       (effects (font (size 1.27 1.27)) hide)
     )
@@
       (effects (font (size 1.27 1.27)) (justify left))
     )
-    (property "Footprint" "Capacitor_SMD:C_0402_1005Metric_Pad0.74x0.62mm_HandSolder" (id 2) (at 92.4052 90.17 0)
+    (property "Footprint" "Capacitor_SMD:C_0402_1005Metric" (id 2) (at 92.4052 90.17 0)
       (effects (font (size 1.27 1.27)) hide)
     )
@@
     (property "Reference" "R15" (id 0) (at 83.82 191.135 90))
     (property "Value" "1k" (id 1) (at 83.82 193.675 90))
-    (property "Footprint" "Resistor_SMD:R_0402_1005Metric_Pad0.72x0.64mm_HandSolder" (id 2) (at 83.82 189.738 90)
+    (property "Footprint" "Resistor_SMD:R_0402_1005Metric" (id 2) (at 83.82 189.738 90)
       (effects (font (size 1.27 1.27)) hide)
     )
@@
     (property "Reference" "R12" (id 0) (at 93.98 147.32 90))
     (property "Value" "1k" (id 1) (at 93.98 149.86 90))
-    (property "Footprint" "Resistor_SMD:R_0402_1005Metric_Pad0.72x0.64mm_HandSolder" (id 2) (at 93.98 155.448 90)
+    (property "Footprint" "Resistor_SMD:R_0402_1005Metric" (id 2) (at 93.98 155.448 90)
       (effects (font (size 1.27 1.27)) hide)
     )
@@
       (effects (font (size 1.27 1.27)) (justify right))
     )
-    (property "Footprint" "LED_SMD:LED_0603_1608Metric_Pad1.05x0.95mm_HandSolder" (id 2) (at 149.86 103.505 0)
+    (property "Footprint" "LED_SMD:LED_0603_1608Metric" (id 2) (at 149.86 103.505 0)
       (effects (font (size 1.27 1.27)) hide)
     )
@@
       (effects (font (size 1.27 1.27)) (justify left))
     )
-    (property "Footprint" "Capacitor_SMD:C_0402_1005Metric_Pad0.74x0.62mm_HandSolder" (id 2) (at 68.2752 52.07 0)
+    (property "Footprint" "Capacitor_SMD:C_0402_1005Metric" (id 2) (at 68.2752 52.07 0)
       (effects (font (size 1.27 1.27)) hide)
     )
@@
     (property "Reference" "R16" (id 0) (at 87.63 219.71 90))
     (property "Value" "1k" (id 1) (at 87.63 222.25 90))
-    (property "Footprint" "Resistor_SMD:R_0402_1005Metric_Pad0.72x0.64mm_HandSolder" (id 2) (at 87.63 227.838 90)
+    (property "Footprint" "Resistor_SMD:R_0402_1005Metric" (id 2) (at 87.63 227.838 90)
       (effects (font (size 1.27 1.27)) hide)
     )
@@
       (effects (font (size 1.27 1.27)) (justify left))
     )
-    (property "Footprint" "Capacitor_SMD:C_0402_1005Metric_Pad0.74x0.62mm_HandSolder" (id 2) (at 113.9952 52.07 0)
+    (property "Footprint" "Capacitor_SMD:C_0402_1005Metric" (id 2) (at 113.9952 52.07 0)
       (effects (font (size 1.27 1.27)) hide)
     )
@@
       (effects (font (size 1.27 1.27)) (justify left))
     )
-    (property "Footprint" "Capacitor_SMD:C_0402_1005Metric_Pad0.74x0.62mm_HandSolder" (id 2) (at 102.5652 52.07 0)
+    (property "Footprint" "Capacitor_SMD:C_0402_1005Metric" (id 2) (at 102.5652 52.07 0)
       (effects (font (size 1.27 1.27)) hide)
     )
@@
       (effects (font (size 1.27 1.27)) (justify left))
     )
-    (property "Footprint" "Resistor_SMD:R_0402_1005Metric_Pad0.72x0.64mm_HandSolder" (id 2) (at 148.082 111.125 90)
+    (property "Footprint" "Resistor_SMD:R_0402_1005Metric" (id 2) (at 148.082 111.125 90)
       (effects (font (size 1.27 1.27)) hide)
     )
@@
     (property "Reference" "FB1" (id 0) (at 189.8142 40.005 90))
     (property "Value" "FerriteBead" (id 1) (at 189.8142 42.545 90))
-    (property "Footprint" "Resistor_SMD:R_0402_1005Metric_Pad0.72x0.64mm_HandSolder" (id 2) (at 189.865 50.038 90)
+    (property "Footprint" "Resistor_SMD:R_0402_1005Metric" (id 2) (at 189.865 50.038 90)
       (effects (font (size 1.27 1.27)) hide)
     )
@@
       (effects (font (size 1.27 1.27)) (justify left))
     )
-    (property "Footprint" "Capacitor_SMD:C_0402_1005Metric_Pad0.74x0.62mm_HandSolder" (id 2) (at 79.7052 52.07 0)
+    (property "Footprint" "Capacitor_SMD:C_0402_1005Metric" (id 2) (at 79.7052 52.07 0)
       (effects (font (size 1.27 1.27)) hide)
     )
@@
       (effects (font (size 1.27 1.27)) (justify left))
     )
-    (property "Footprint" "Capacitor_SMD:C_0402_1005Metric_Pad0.74x0.62mm_HandSolder" (id 2) (at 56.8452 52.07 0)
+    (property "Footprint" "Capacitor_SMD:C_0402_1005Metric" (id 2) (at 56.8452 52.07 0)
       (effects (font (size 1.27 1.27)) hide)
     )
@@
       (effects (font (size 1.27 1.27)) (justify left))
     )
-    (property "Footprint" "Capacitor_SMD:C_0402_1005Metric_Pad0.74x0.62mm_HandSolder" (id 2) (at 103.8352 90.17 0)
+    (property "Footprint" "Capacitor_SMD:C_0402_1005Metric" (id 2) (at 103.8352 90.17 0)
       (effects (font (size 1.27 1.27)) hide)
     )
@@
       (effects (font (size 1.27 1.27)) (justify left))
     )
-    (property "Footprint" "Resistor_SMD:R_0402_1005Metric_Pad0.72x0.64mm_HandSolder" (id 2) (at 106.807 147.955 90)
+    (property "Footprint" "Resistor_SMD:R_0402_1005Metric" (id 2) (at 106.807 147.955 90)
       (effects (font (size 1.27 1.27)) hide)
     )
@@
       (effects (font (size 1.27 1.27)) (justify left))
     )
-    (property "Footprint" "Capacitor_SMD:C_0402_1005Metric_Pad0.74x0.62mm_HandSolder" (id 2) (at 274.6502 58.42 0)
+    (property "Footprint" "Capacitor_SMD:C_0402_1005Metric" (id 2) (at 274.6502 58.42 0)
       (effects (font (size 1.27 1.27)) hide)
     )
@@
       (effects (font (size 1.27 1.27)) (justify left))
     )
-    (property "Footprint" "Capacitor_SMD:C_0603_1608Metric_Pad1.08x0.95mm_HandSolder" (id 2) (at 103.8352 111.76 0)
+    (property "Footprint" "Capacitor_SMD:C_0603_1608Metric" (id 2) (at 103.8352 111.76 0)
       (effects (font (size 1.27 1.27)) hide)
     )
@@
       (effects (font (size 1.27 1.27)) (justify left))
     )
-    (property "Footprint" "Capacitor_SMD:C_0402_1005Metric_Pad0.74x0.62mm_HandSolder" (id 2) (at 68.9102 233.68 0)
+    (property "Footprint" "Capacitor_SMD:C_0402_1005Metric" (id 2) (at 68.9102 233.68 0)
       (effects (font (size 1.27 1.27)) hide)
     )
@@
       (effects (font (size 1.27 1.27)) (justify left))
     )
-    (property "Footprint" "Capacitor_SMD:C_0402_1005Metric_Pad0.74x0.62mm_HandSolder" (id 2) (at 241.6302 58.42 0)
+    (property "Footprint" "Capacitor_SMD:C_0402_1005Metric" (id 2) (at 241.6302 58.42 0)
       (effects (font (size 1.27 1.27)) hide)
     )
@@
       (effects (font (size 1.27 1.27)) (justify left))
     )
-    (property "Footprint" "Resistor_SMD:R_0402_1005Metric_Pad0.72x0.64mm_HandSolder" (id 2) (at 344.932 55.88 90)
+    (property "Footprint" "Resistor_SMD:R_0402_1005Metric" (id 2) (at 344.932 55.88 90)
       (effects (font (size 1.27 1.27)) hide)
     )
@@
       (effects (font (size 1.27 1.27)) (justify left))
     )
-    (property "Footprint" "Capacitor_SMD:C_0603_1608Metric_Pad1.08x0.95mm_HandSolder" (id 2) (at 45.4152 73.66 0)
+    (property "Footprint" "Capacitor_SMD:C_0603_1608Metric" (id 2) (at 45.4152 73.66 0)
       (effects (font (size 1.27 1.27)) hide)
     )
@@
       (effects (font (size 1.27 1.27)) (justify left))
     )
-    (property "Footprint" "Capacitor_SMD:C_0402_1005Metric_Pad0.74x0.62mm_HandSolder" (id 2) (at 68.9102 215.9 0)
+    (property "Footprint" "Capacitor_SMD:C_0402_1005Metric" (id 2) (at 68.9102 215.9 0)
       (effects (font (size 1.27 1.27)) hide)
     )
@@
     (property "Reference" "R14" (id 0) (at 69.85 182.88 90))
     (property "Value" "27.4" (id 1) (at 69.85 184.785 90))
-    (property "Footprint" "Resistor_SMD:R_0402_1005Metric_Pad0.72x0.64mm_HandSolder" (id 2) (at 69.85 182.118 90)
-      (effects (font (size 1.27 1.27)) hide)
-    )
+    (property "Footprint" "Resistor_SMD:R_0402_1005Metric" (id 2) (at 69.85 182.118 90)
+      (effects (font (size 1.27 1.27)) hide)
+    )
